Commit message: Add gmapping localisation

File: Raspberry/src/robot_description/urdf/robot.xacro (robot description, xacro)
@@ -99,5 +99,5 @@
     <joint name="hokuyo_joint" type="fixed">
         <axis xyz="0 1 0" />
-        <origin xyz="${-cameraSize+chassisLength/2} 0 ${cameraSize+wheelRadius+cameraSize/2}" rpy="0 0 0"/>
+        <origin xyz="${-cameraSize+chassisLength/2} 0 ${2*wheelRadius}" rpy="0 0 0"/>
         <parent link="chassis"/>
         <child link="hokuyo_link"/>

Commit message: Add table urdf description

File: Raspberry/src/robot_description/urdf/robot.xacro (robot description, xacro)
@@ -3,13 +3,13 @@
   <xacro:property name="PI" value="3.1415926535897931"/>
   <xacro:property name="chassisHeight" value="0.1"/>
-  <xacro:property name="chassisLength" value="0.4"/>
+  <xacro:property name="chassisLength" value="0.3"/>
   <xacro:property name="chassisWidth" value="0.2"/>
-  <xacro:property name="chassisMass" value="50"/>
+  <xacro:property name="chassisMass" value="5"/>
   <xacro:property name="casterRadius" value="0.05"/>
-  <xacro:property name="casterMass" value="5"/>
+  <xacro:property name="casterMass" value="0.5"/>
   <xacro:property name="wheelWidth" value="0.05"/>
   <xacro:property name="wheelRadius" value="0.1"/>
   <xacro:property name="wheelPos" value="0.2"/>
-  <xacro:property name="wheelMass" value="5"/>
+  <xacro:property name="wheelMass" value="0.5"/>
   <xacro:property name="cameraSize" value="0.05"/>
   <xacro:property name="cameraMass" value="0.1"/>
