Commit message: Untabify code

File: Raspberry/src/robot_description/urdf/macros.xacro (robot description, xacro)
@@ -1,64 +1,64 @@
 <?xml version="1.0"?>
 <robot>
-    <macro name="cylinder_inertia" params="m r h">
-        <inertia ixx="${m*(3*r*r+h*h)/12}" ixy = "0" ixz = "0"
-                 iyy="${m*(3*r*r+h*h)/12}" iyz = "0"
-                 izz="${m*r*r/2}" />
-    </macro>
-    <macro name="box_inertia" params="m x y z">
-        <inertia ixx="${m*(y*y+z*z)/12}" ixy = "0" ixz = "0"
-                 iyy="${m*(x*x+z*z)/12}" iyz = "0"
-                 izz="${m*(x*x+z*z)/12}" />
-    </macro>
-    <macro name="sphere_inertia" params="m r">
-        <inertia ixx="${2*m*r*r/5}" ixy = "0" ixz = "0"
-                 iyy="${2*m*r*r/5}" iyz = "0"
-                 izz="${2*m*r*r/5}" />
-    </macro>
-    <macro name="wheel" params="lr tY">
-        <link name="${lr}_wheel">
-            <collision>
-                <origin xyz="0 0 0" rpy="0 ${PI/2} ${PI/2}" />
-                <geometry>
-                <cylinder length="${wheelWidth}" radius="${wheelRadius}"/>
-                </geometry>
-            </collision>
-            <visual>
-                <origin xyz="0 0 0" rpy="0 ${PI/2} ${PI/2}" />
-                <geometry>
-                <cylinder length="${wheelWidth}" radius="${wheelRadius}"/>
-                </geometry>
-                <material name="black"/>
-            </visual>
-            <inertial>
-                <origin xyz="0 0 0" rpy="0 ${PI/2} ${PI/2}" />
-                <mass value="${wheelMass}"/>
-                <cylinder_inertia m="${wheelMass}" r="${wheelRadius}" h="${wheelWidth}"/>
-            </inertial>
-        </link>
-        <gazebo reference="${lr}_wheel">
-            <mu1 value="1.0"/>
-            <mu2 value="1.0"/>
-            <kp  value="10000000.0" />
-            <kd  value="1.0" />
-            <fdir1 value="1 0 0"/>
-            <material>Gazebo/Black</material>
-        </gazebo>
-        <joint name="${lr}_wheel_hinge" type="continuous">
-            <parent link="chassis"/>
-            <child link="${lr}_wheel"/>
-            <origin xyz="${+wheelPos-chassisLength/4} ${tY*wheelWidth/2+tY*chassisWidth/2} ${wheelRadius}" rpy="0 0 0" />
-            <axis xyz="0 1 0" rpy="0 0 0" />
-            <limit effort="100" velocity="100"/>
-            <joint_properties damping="0.0" friction="0.0"/>
-        </joint>
-        <transmission name="${lr}_trans">
-            <type>transmission_interface/SimpleTransmission</type>
-            <joint name="${lr}_wheel_hinge"/>
-            <actuator name="${lr}Motor">
-                <hardwareInterface>EffortJointInterface</hardwareInterface>
-                <mechanicalReduction>10</mechanicalReduction>
-            </actuator>
-        </transmission>
-    </macro>
+  <macro name="cylinder_inertia" params="m r h">
+    <inertia ixx="${m*(3*r*r+h*h)/12}" ixy = "0" ixz = "0"
+             iyy="${m*(3*r*r+h*h)/12}" iyz = "0"
+             izz="${m*r*r/2}" />
+  </macro>
+  <macro name="box_inertia" params="m x y z">
+    <inertia ixx="${m*(y*y+z*z)/12}" ixy = "0" ixz = "0"
+             iyy="${m*(x*x+z*z)/12}" iyz = "0"
+             izz="${m*(x*x+z*z)/12}" />
+  </macro>
+  <macro name="sphere_inertia" params="m r">
+    <inertia ixx="${2*m*r*r/5}" ixy = "0" ixz = "0"
+             iyy="${2*m*r*r/5}" iyz = "0"
+             izz="${2*m*r*r/5}" />
+  </macro>
+  <macro name="wheel" params="lr tY">
+    <link name="${lr}_wheel">
+      <collision>
+        <origin xyz="0 0 0" rpy="0 ${PI/2} ${PI/2}" />
+        <geometry>
+        <cylinder length="${wheelWidth}" radius="${wheelRadius}"/>
+        </geometry>
+      </collision>
+      <visual>
+        <origin xyz="0 0 0" rpy="0 ${PI/2} ${PI/2}" />
+        <geometry>
+        <cylinder length="${wheelWidth}" radius="${wheelRadius}"/>
+        </geometry>
+        <material name="black"/>
+      </visual>
+      <inertial>
+        <origin xyz="0 0 0" rpy="0 ${PI/2} ${PI/2}" />
+        <mass value="${wheelMass}"/>
+        <cylinder_inertia m="${wheelMass}" r="${wheelRadius}" h="${wheelWidth}"/>
+      </inertial>
+    </link>
+    <gazebo reference="${lr}_wheel">
+      <mu1 value="1.0"/>
+      <mu2 value="1.0"/>
+      <kp value="10000000.0" />
+      <kd value="1.0" />
+      <fdir1 value="1 0 0"/>
+      <material>Gazebo/Black</material>
+    </gazebo>
+    <joint name="${lr}_wheel_hinge" type="continuous">
+      <parent link="chassis"/>
+      <child link="${lr}_wheel"/>
+      <origin xyz="${+wheelPos-chassisLength/4} ${tY*wheelWidth/2+tY*chassisWidth/2} ${wheelRadius}" rpy="0 0 0" />
+      <axis xyz="0 1 0" rpy="0 0 0" />
+      <limit effort="100" velocity="100"/>
+      <joint_properties damping="0.0" friction="0.0"/>
+    </joint>
+    <transmission name="${lr}_trans">
+      <type>transmission_interface/SimpleTransmission</type>
+      <joint name="${lr}_wheel_hinge"/>
+      <actuator name="${lr}Motor">
+        <hardwareInterface>EffortJointInterface</hardwareInterface>
+        <mechanicalReduction>10</mechanicalReduction>
+      </actuator>
+    </transmission>
+  </macro>
 </robot>

File: Raspberry/src/robot_description/urdf/materials.xacro (robot description, xacro)
@@ -1,27 +1,27 @@
 <?xml version="1.0"?>
 <robot>
-    <material name="black">
-        <color rgba="0.0 0.0 0.0 1.0"/>
-    </material>
-    <material name="blue">
-        <color rgba="0.0 0.0 0.8 1.0"/>
-    </material>
-    <material name="green">
-        <color rgba="0.0 0.8 0.0 1.0"/>
-    </material>
-    <material name="grey">
-        <color rgba="0.2 0.2 0.2 1.0"/>
-    </material>
-    <material name="orange">
-        <color rgba="${255/255} ${108/255} ${10/255} 1.0"/>
-    </material>
-    <material name="brown">
-        <color rgba="${222/255} ${207/255} ${195/255} 1.0"/>
-    </material>
-    <material name="red">
-        <color rgba="0.8 0.0 0.0 1.0"/>
-    </material>
-    <material name="white">
-        <color rgba="1.0 1.0 1.0 1.0"/>
-    </material>
+  <material name="black">
+    <color rgba="0.0 0.0 0.0 1.0"/>
+  </material>
+  <material name="blue">
+    <color rgba="0.0 0.0 0.8 1.0"/>
+  </material>
+  <material name="green">
+    <color rgba="0.0 0.8 0.0 1.0"/>
+  </material>
+  <material name="grey">
+    <color rgba="0.2 0.2 0.2 1.0"/>
+  </material>
+  <material name="orange">
+    <color rgba="${255/255} ${108/255} ${10/255} 1.0"/>
+  </material>
+  <material name="brown">
+    <color rgba="${222/255} ${207/255} ${195/255} 1.0"/>
+  </material>
+  <material name="red">
+    <color rgba="0.8 0.0 0.0 1.0"/>
+  </material>
+  <material name="white">
+    <color rgba="1.0 1.0 1.0 1.0"/>
+  </material>
 </robot>

File: Raspberry/src/robot_description/urdf/robot.xacro (robot description, xacro)
@@ -1,124 +1,124 @@
 <?xml version="1.0"?>
 <robot name="robot" xmlns:xacro="http://www.ros.org/wiki/xacro">
-    <xacro:property name="PI" value="3.1415926535897931"/>
-    <xacro:property name="chassisHeight" value="0.1"/>
-    <xacro:property name="chassisLength" value="0.4"/>
-    <xacro:property name="chassisWidth" value="0.2"/>
-    <xacro:property name="chassisMass" value="50"/>
-    <xacro:property name="casterRadius" value="0.05"/>
-    <xacro:property name="casterMass" value="5"/>
-    <xacro:property name="wheelWidth" value="0.05"/>
-    <xacro:property name="wheelRadius" value="0.1"/>
-    <xacro:property name="wheelPos" value="0.2"/>
-    <xacro:property name="wheelMass" value="5"/>
-    <xacro:property name="cameraSize" value="0.05"/>
-    <xacro:property name="cameraMass" value="0.1"/>
-    <xacro:include filename="$(find robot_description)/urdf/robot.gazebo" />
-    <xacro:include filename="$(find robot_description)/urdf/materials.xacro" />
-    <xacro:include filename="$(find robot_description)/urdf/macros.xacro" />
-    <!-- Chassis -->
-    <link name="footprint" />
-    <joint name="base_joint" type="fixed">
-        <parent link="footprint"/>
-        <child link="chassis"/>
-    </joint>
-    <link name="chassis">
-        <collision>
-            <origin xyz="0 0 ${wheelRadius}" rpy="0 0 0"/>
-            <geometry>
-                <box size="${chassisLength} ${chassisWidth} ${chassisHeight}"/>
-            </geometry>
-        </collision>
-        <visual>
-            <origin xyz="0 0 ${wheelRadius}" rpy="0 0 0"/>
-            <geometry>
-                <box size="${chassisLength} ${chassisWidth} ${chassisHeight}"/>
-            </geometry>
-            <material name="orange"/>
-        </visual>
-        <inertial>
-            <origin xyz="0 0 ${wheelRadius}" rpy="0 0 0"/>
-            <mass value="${chassisMass}"/>
-            <box_inertia m="${chassisMass}" x="${chassisLength}" y="${chassisWidth}" z="${chassisHeight}"/>
-        </inertial>
-    </link>
-    <!-- Caster wheel -->
-    <joint name="fixed" type="fixed">
-        <parent link="chassis"/>
-        <child link="caster_wheel"/>
-    </joint>
-    <link name="caster_wheel">
-        <collision>
-            <origin xyz="${casterRadius-chassisLength/2} 0 ${casterRadius-chassisHeight+wheelRadius}" rpy="0 0 0"/>
-            <geometry>
-                <sphere radius="${casterRadius}"/>
-            </geometry>
-        </collision>
-        <visual>
-            <origin xyz="${casterRadius-chassisLength/2} 0 ${casterRadius-chassisHeight+wheelRadius}" rpy="0 0 0"/>
-            <geometry>
-                <sphere radius="${casterRadius}"/>
-            </geometry>
-        </visual>
-        <inertial>
-            <origin xyz="${casterRadius-chassisLength/2} 0 ${casterRadius-chassisHeight+wheelRadius}" rpy="0 0 0"/>
-            <mass value="${casterMass}"/>
-            <sphere_inertia m="${casterMass}" r="${casterRadius}"/>
-        </inertial>
-    </link>
-    <!-- Fixed wheels -->
-    <wheel lr="left" tY="1"/>
-    <wheel lr="right" tY="-1"/>
-    <!-- Camera -->
-    <joint name="camera_joint" type="fixed">
-        <origin xyz="${-cameraSize+chassisLength/2} 0 ${cameraSize+wheelRadius+cameraSize/2+0.08}" rpy="0 0 0"/>
-        <parent link="chassis"/>
-        <child link="camera"/>
-    </joint>
-    <link name="camera">
-        <collision>
-            <origin xyz="0 0 0" rpy="0 0 0"/>
-            <geometry>
-                <box size="${cameraSize} ${cameraSize} ${cameraSize}"/>
-            </geometry>
-        </collision>
-        <visual>
-            <origin xyz="0 0 0" rpy="0 0 0"/>
-            <geometry>
-                <box size="${cameraSize} ${cameraSize} ${cameraSize}"/>
-            </geometry>
-            <material name="blue"/>
-        </visual>
-        <inertial>
-            <mass value="${cameraMass}" />
-            <origin xyz="0 0 0" rpy="0 0 0"/>
-            <box_inertia m="${cameraMass}" x="${cameraSize}" y="${cameraSize}" z="${cameraSize}" />
-        </inertial>
-    </link>
-    <!-- Hokuyo -->
-    <joint name="hokuyo_joint" type="fixed">
-        <axis xyz="0 1 0" />
-        <origin xyz="${-cameraSize+chassisLength/2} 0 ${2*wheelRadius}" rpy="0 0 0"/>
-        <parent link="chassis"/>
-        <child link="hokuyo_link"/>
-    </joint>
-    <link name="hokuyo_link">
-        <collision>
-            <origin xyz="0 0 0" rpy="0 0 0"/>
-            <geometry>
-                <box size="0.1 0.1 0.1"/>
-            </geometry>
-        </collision>
-        <visual>
-            <origin xyz="0 0 0" rpy="0 0 0"/>
-            <geometry>
-                <mesh filename="package://robot_description/urdf/hokuyo.dae"/>
-            </geometry>
-        </visual>
-        <inertial>
-            <mass value="1e-5" />
-            <origin xyz="0 0 0" rpy="0 0 0"/>
-            <inertia ixx="1e-6" ixy="0" ixz="0" iyy="1e-6" iyz="0" izz="1e-6" />
-        </inertial>
-    </link>
+  <xacro:property name="PI" value="3.1415926535897931"/>
+  <xacro:property name="chassisHeight" value="0.1"/>
+  <xacro:property name="chassisLength" value="0.4"/>
+  <xacro:property name="chassisWidth" value="0.2"/>
+  <xacro:property name="chassisMass" value="50"/>
+  <xacro:property name="casterRadius" value="0.05"/>
+  <xacro:property name="casterMass" value="5"/>
+  <xacro:property name="wheelWidth" value="0.05"/>
+  <xacro:property name="wheelRadius" value="0.1"/>
+  <xacro:property name="wheelPos" value="0.2"/>
+  <xacro:property name="wheelMass" value="5"/>
+  <xacro:property name="cameraSize" value="0.05"/>
+  <xacro:property name="cameraMass" value="0.1"/>
+  <xacro:include filename="$(find robot_description)/urdf/robot.gazebo" />
+  <xacro:include filename="$(find robot_description)/urdf/materials.xacro" />
+  <xacro:include filename="$(find robot_description)/urdf/macros.xacro" />
+  <!-- Chassis -->
+  <link name="footprint" />
+  <joint name="base_joint" type="fixed">
+    <parent link="footprint"/>
+    <child link="chassis"/>
+  </joint>
+  <link name="chassis">
+    <collision>
+      <origin xyz="0 0 ${wheelRadius}" rpy="0 0 0"/>
+      <geometry>
+        <box size="${chassisLength} ${chassisWidth} ${chassisHeight}"/>
+      </geometry>
+    </collision>
+    <visual>
+      <origin xyz="0 0 ${wheelRadius}" rpy="0 0 0"/>
+      <geometry>
+        <box size="${chassisLength} ${chassisWidth} ${chassisHeight}"/>
+      </geometry>
+      <material name="orange"/>
+    </visual>
+    <inertial>
+      <origin xyz="0 0 ${wheelRadius}" rpy="0 0 0"/>
+      <mass value="${chassisMass}"/>
+      <box_inertia m="${chassisMass}" x="${chassisLength}" y="${chassisWidth}" z="${chassisHeight}"/>
+    </inertial>
+  </link>
+  <!-- Caster wheel -->
+  <joint name="fixed" type="fixed">
+    <parent link="chassis"/>
+    <child link="caster_wheel"/>
+  </joint>
+  <link name="caster_wheel">
+    <collision>
+      <origin xyz="${casterRadius-chassisLength/2} 0 ${casterRadius-chassisHeight+wheelRadius}" rpy="0 0 0"/>
+      <geometry>
+        <sphere radius="${casterRadius}"/>
+      </geometry>
+    </collision>
+    <visual>
+      <origin xyz="${casterRadius-chassisLength/2} 0 ${casterRadius-chassisHeight+wheelRadius}" rpy="0 0 0"/>
+      <geometry>
+        <sphere radius="${casterRadius}"/>
+      </geometry>
+    </visual>
+    <inertial>
+      <origin xyz="${casterRadius-chassisLength/2} 0 ${casterRadius-chassisHeight+wheelRadius}" rpy="0 0 0"/>
+      <mass value="${casterMass}"/>
+      <sphere_inertia m="${casterMass}" r="${casterRadius}"/>
+    </inertial>
+  </link>
+  <!-- Fixed wheels -->
+  <wheel lr="left" tY="1"/>
+  <wheel lr="right" tY="-1"/>
+  <!-- Camera -->
+  <joint name="camera_joint" type="fixed">
+    <origin xyz="${-cameraSize+chassisLength/2} 0 ${cameraSize+wheelRadius+cameraSize/2+0.08}" rpy="0 0 0"/>
+    <parent link="chassis"/>
+    <child link="camera"/>
+  </joint>
+  <link name="camera">
+    <collision>
+      <origin xyz="0 0 0" rpy="0 0 0"/>
+      <geometry>
+        <box size="${cameraSize} ${cameraSize} ${cameraSize}"/>
+      </geometry>
+    </collision>
+    <visual>
+      <origin xyz="0 0 0" rpy="0 0 0"/>
+      <geometry>
+        <box size="${cameraSize} ${cameraSize} ${cameraSize}"/>
+      </geometry>
+      <material name="blue"/>
+    </visual>
+    <inertial>
+      <mass value="${cameraMass}" />
+      <origin xyz="0 0 0" rpy="0 0 0"/>
+      <box_inertia m="${cameraMass}" x="${cameraSize}" y="${cameraSize}" z="${cameraSize}" />
+    </inertial>
+  </link>
+  <!-- Hokuyo -->
+  <joint name="hokuyo_joint" type="fixed">
+    <axis xyz="0 1 0" />
+    <origin xyz="${-cameraSize+chassisLength/2} 0 ${2*wheelRadius}" rpy="0 0 0"/>
+    <parent link="chassis"/>
+    <child link="hokuyo_link"/>
+  </joint>
+  <link name="hokuyo_link">
+    <collision>
+      <origin xyz="0 0 0" rpy="0 0 0"/>
+      <geometry>
+        <box size="0.1 0.1 0.1"/>
+      </geometry>
+    </collision>
+    <visual>
+      <origin xyz="0 0 0" rpy="0 0 0"/>
+      <geometry>
+        <mesh filename="package://robot_description/urdf/hokuyo.dae"/>
+      </geometry>
+    </visual>
+    <inertial>
+      <mass value="1e-5" />
+      <origin xyz="0 0 0" rpy="0 0 0"/>
+      <inertia ixx="1e-6" ixy="0" ixz="0" iyy="1e-6" iyz="0" izz="1e-6" />
+    </inertial>
+  </link>
 </robot>

Commit message: Fix simulated robot model, add amcl

File: Raspberry/src/robot_description/urdf/macros.xacro (robot description, xacro)
@@ -48,5 +48,5 @@
       <parent link="chassis"/>
       <child link="${lr}_wheel"/>
-      <origin xyz="${+wheelPos-chassisLength/4} ${tY*wheelWidth/2+tY*chassisWidth/2} ${wheelRadius}" rpy="0 0 0" />
+      <origin xyz="${-wheelPos} ${tY*wheelWidth/2+tY*chassisWidth/2} ${wheelRadius}" rpy="0 0 0" />
       <axis xyz="0 1 0" rpy="0 0 0" />
       <limit effort="100" velocity="100"/>

File: Raspberry/src/robot_description/urdf/robot.xacro (robot description, xacro)
@@ -8,7 +8,8 @@
   <xacro:property name="casterRadius" value="0.05"/>
   <xacro:property name="casterMass" value="0.5"/>
+  <xacro:property name="casterPos" value="0.2"/>
   <xacro:property name="wheelWidth" value="0.05"/>
   <xacro:property name="wheelRadius" value="0.1"/>
-  <xacro:property name="wheelPos" value="0.2"/>
+  <xacro:property name="wheelPos" value="0.05"/>  <!-- Distance of the wheels axis to the center of the robot -->
   <xacro:property name="wheelMass" value="0.5"/>
   <xacro:property name="cameraSize" value="0.05"/>
@@ -18,8 +19,9 @@
   <xacro:include filename="$(find robot_description)/urdf/macros.xacro" />
   <!-- Chassis -->
-  <link name="footprint" />
+  <link name="base_link" />
   <joint name="base_joint" type="fixed">
-    <parent link="footprint"/>
+    <parent link="base_link"/>
     <child link="chassis"/>
+    <origin xyz="${wheelPos} 0 0" rpy="0 0 0" />
   </joint>
   <link name="chassis">
@@ -47,4 +49,5 @@
     <parent link="chassis"/>
     <child link="caster_wheel"/>
+    <origin xyz="${casterPos} 0 0" rpy="0 0 0" />
   </joint>
   <link name="caster_wheel">
@@ -98,6 +101,5 @@
   <!-- Hokuyo -->
   <joint name="hokuyo_joint" type="fixed">
-    <axis xyz="0 1 0" />
-    <origin xyz="${-cameraSize+chassisLength/2} 0 ${2*wheelRadius}" rpy="0 0 0"/>
+    <origin xyz="${-cameraSize+chassisLength/2} 0 ${2*wheelRadius + 0.01}" rpy="0 0 0"/>
     <parent link="chassis"/>
     <child link="hokuyo_link"/>
@@ -111,5 +113,5 @@
     </collision>
     <visual>
-      <origin xyz="0 0 0" rpy="0 0 0"/>
+      <origin xyz="0 0 -0.02" rpy="0 0 0"/>
       <geometry>
         <mesh filename="package://robot_description/urdf/hokuyo.dae"/>
